File: pcb/proto-nrf-hat/proto.kicad_pcb (KiCad board)
At the start: 2 copper layers, 54.9 x 48 mm, 15 parts, among them J1 Servo 1, J11 Sensors, J12 Conn_01x02, J2 Power/i2c, J3 Port B, J4 Port C, J5 Port D, J6 Servo 2, J7 Servo 3, J8 Conn_02x04_Counter_Clockwise, U1 MCP1700-3302E_TO92

Commit message: sensors working and stuff
Parts:
- U1: value MCP1700-3302E_TO92 -> LP2950-3.0_TO92
- moved U1 5.58 mm to (194.8, 113.8)
- moved J11 4.23 mm to (202.7, 119.9)
- moved J8 2.54 mm to (178.6, 100.6)
- moved J1 1.02 mm to (200.2, 96.8)
- moved J6 1.02 mm to (200.2, 100.6)
- moved J7 1.02 mm to (200.2, 104.4)
Connections:
- J3 pad 2: /CSN -> /CE
- J3 pad 3: /CE -> Net-(J3-Pad3)
- J4 pad 4: /SDA -> (no net)
- J4 pad 5: /SCL -> /SDA
- J4 pad 6: (no net) -> /SCL
- J8 pad 4: /CSN -> Net-(J3-Pad3)
- U1 pad 1: Earth -> /Reg3v
- U1 pad 2: +5V -> Earth
- U1 pad 3: /Reg3v -> +5V
Routing:
- net Earth: track 130.1 -> 85.3 mm, vias 2 -> 4
- net /CSN: track 21.2 -> 0.00 mm
- net Net-(J3-Pad3): track 0.00 -> 12.8 mm
- net /SCL: track 14.1 -> 25.7 mm
- net /Reg3v: track 47.2 -> 35.7 mm
- net +5V: track 58.0 -> 51.6 mm
- net /MOSI: track 20.9 -> 17.6 mm
- net /CE: track 18.7 -> 22.1 mm
- net /MISO: track 42.1 -> 44.7 mm
- net Net-(J1-Pad1): track 7.48 -> 5.91 mm
- net /SCK: track 56.9 -> 55.6 mm
- net /SDA: track 22.3 -> 21.1 mm
- net /IRQ: track 12.9 -> 14.0 mm
- net Net-(J4-Pad3): track 11.4 -> 10.8 mm
- net Net-(J4-Pad2): track 12.0 -> 12.5 mm
- removed copper zone on B.Cu, net Earth
Other:
- board size 54.9 x 48 mm -> 53.6 x 47.2 mm
