File: pcb/proto-nrf-hat/proto.sch (KiCad schematic (older format))
At the start: 17 parts, among them J1 Servo 1, J10 Conn_01x01, J11 Sensors, J12 Conn_01x02, J2 Power/i2c, J3 Port B, J4 Port C, J5 Port D, J6 Servo 2, J7 Servo 3, J8 Conn_02x04_Counter_Clockwise, J9 Conn_01x01, U1 MCP1700-3302E_TO92

Commit message: sensors working and stuff
Parts:
- removed U1: MCP1700-3302E_TO92, TO_SOT_Packages_THT:TO-92_Inline_Wide, symbol MCP1700-3302E_TO92
- added U1: LP2950-3.0_TO92, TO_SOT_Packages_THT:TO-92_Inline_Wide, symbol LP2950-3.0_TO92
Connections:
- net +5V: now also U1.3 (VI)
- net CE: now also J3.2 (Pin_2); no longer J3.3 (Pin_3)
- net CSN: no longer J3.2 (Pin_2), J8.4 (Pin_4)
- net Earth: now also U1.2 (GND)
- net Reg3v: now also U1.1 (VO)
- net SCL: now also J4.6 (Pin_6); no longer J4.5 (Pin_5)
- net SDA: now also J4.5 (Pin_5); no longer J4.4 (Pin_4)
- new net: J3.3 (Pin_3), J8.4 (Pin_4)
Other:
- moved on the sheet: C1, C2
Changed lines of the file:
@@
-$EndComp
-$Comp
-L MCP1700-3302E_TO92 U1
-U 1 1 5BBB6989
-P 4950 2100
-F 0 "U1" H 4800 1975 50  0000 C CNN
-F 1 "MCP1700-3302E_TO92" H 4950 1975 50  0000 L CNN
-F 2 "TO_SOT_Packages_THT:TO-92_Inline_Wide" H 4950 1900 50  0001 C CIN
-F 3 "" H 4950 2100 50  0001 C CNN
-	1    4950 2100
-	1    0    0    -1
 $EndComp
 $Comp
@@
 L +5V #PWR010
 U 1 1 5BBB7322
-P 4450 2100
-F 0 "#PWR010" H 4450 1950 50  0001 C CNN
-F 1 "+5V" H 4450 2240 50  0000 C CNN
-F 2 "" H 4450 2100 50  0001 C CNN
-F 3 "" H 4450 2100 50  0001 C CNN
-	1    4450 2100
+P 4450 1700
+F 0 "#PWR010" H 4450 1550 50  0001 C CNN
+F 1 "+5V" H 4450 1840 50  0000 C CNN
+F 2 "" H 4450 1700 50  0001 C CNN
+F 3 "" H 4450 1700 50  0001 C CNN
+	1    4450 1700
 	0    -1   -1   0
 $EndComp
@@
 L Earth #PWR011
 U 1 1 5BBB7616
-P 4950 1550
-F 0 "#PWR011" H 4950 1300 50  0001 C CNN
-F 1 "Earth" H 4950 1400 50  0001 C CNN
-F 2 "" H 4950 1550 50  0001 C CNN
-F 3 "" H 4950 1550 50  0001 C CNN
-	1    4950 1550
+P 4850 1900
+F 0 "#PWR011" H 4850 1650 50  0001 C CNN
+F 1 "Earth" H 4850 1750 50  0001 C CNN
+F 2 "" H 4850 1900 50  0001 C CNN
+F 3 "" H 4850 1900 50  0001 C CNN
+	1    4850 1900
 	-1   0    0    1
-$EndComp
-$Comp
-L CP C1
-U 1 1 5BBB776B
-P 4700 1750
-F 0 "C1" H 4725 1850 50  0000 L CNN
-F 1 "CP" H 4725 1650 50  0000 L CNN
-F 2 "Capacitors_THT:CP_Radial_Tantal_D5.5mm_P5.00mm" H 4738 1600 50  0001 C CNN
-F 3 "" H 4700 1750 50  0001 C CNN
-	1    4700 1750
-	0    -1   -1   0
 $EndComp
 $Comp
 L CP C2
 U 1 1 5BBB7B4C
-P 5200 1750
-F 0 "C2" H 5225 1850 50  0000 L CNN
-F 1 "CP" H 5225 1650 50  0000 L CNN
-F 2 "Capacitors_THT:CP_Radial_Tantal_D5.5mm_P5.00mm" H 5238 1600 50  0001 C CNN
-F 3 "" H 5200 1750 50  0001 C CNN
-	1    5200 1750
+P 5150 2150
+F 0 "C2" H 5175 2250 50  0000 L CNN
+F 1 "CP" H 5175 2050 50  0000 L CNN
+F 2 "Capacitors_THT:CP_Radial_Tantal_D5.5mm_P5.00mm" H 5188 2000 50  0001 C CNN
+F 3 "" H 5150 2150 50  0001 C CNN
+	1    5150 2150
 	0    1    1    0
 $EndComp
@@
 	-1   0    0    1
 $EndComp
-Text Label 5400 2450 0    60   ~ 0
+Text Label 4550 2000 0    60   ~ 0
 +3v
 Text Label 4400 3250 0    60   ~ 0
@@
 Text Label 5400 2800 0    60   ~ 0
 MOSI
-Text Label 5700 2650 0    60   ~ 0
+Text Label 4850 3150 0    60   ~ 0
 CSN
-Text Label 5350 1950 0    60   ~ 0
+Text Label 5350 2000 0    60   ~ 0
 Reg3v
 $Comp
@@
 $EndComp
 Wire Wire Line
-	5250 2100 5350 2100
-Wire Wire Line
-	4450 2100 4650 2100
-Wire Wire Line
-	4950 1800 4950 1550
-Wire Wire Line
-	4850 1750 5050 1750
-Connection ~ 4950 1750
-Wire Wire Line
-	4550 1750 4550 2100
-Connection ~ 4550 2100
-Connection ~ 5350 2100
+	5250 1700 5350 1700
+Wire Wire Line
+	4450 1700 4650 1700
+Connection ~ 4550 1700
+Connection ~ 5350 1700
 Wire Wire Line
 	3300 2550 3400 2550
 Wire Wire Line
+	3400 1750 3800 1750
+Wire Wire Line
+	3300 2450 3550 2450
+Wire Wire Line
+	3550 2450 3550 2200
+Wire Wire Line
+	3550 2200 3800 2200
+Wire Wire Line
+	3300 2350 3500 2350
+Wire Wire Line
+	3500 2350 3500 2650
+Wire Wire Line
+	3500 2650 3800 2650
+Wire Wire Line
+	6100 2550 6050 2550
+Wire Wire Line
+	6050 2550 6050 2400
+Wire Wire Line
+	6050 2100 6050 2050
+Wire Wire Line
+	6050 1750 6050 1650
+Wire Wire Line
+	5750 3250 4350 3250
+Wire Wire Line
+	6000 3050 6100 3050
+Wire Wire Line
+	5650 2950 6100 2950
+Wire Wire Line
+	5250 2800 5900 2800
+Wire Wire Line
+	5900 2850 6100 2850
+Wire Wire Line
+	5900 2800 5900 2850
+Wire Wire Line
+	5750 2650 5750 3250
+Wire Wire Line
+	5350 2500 4600 2500
+Wire Wire Line
+	4600 2500 4600 2700
+Wire Wire Line
+	4600 2700 4750 2700
+Wire Wire Line
+	5350 1700 5350 2500
+Wire Wire Line
+	4350 3250 4350 2800
+Wire Wire Line
+	4350 2800 4750 2800
+Wire Wire Line
+	5700 3050 4750 3050
+Wire Wire Line
+	4750 3050 4750 2900
+Wire Wire Line
+	5650 2950 5650 2700
+Wire Wire Line
+	5650 2700 5250 2700
+Wire Wire Line
+	6500 4000 5350 4000
+Wire Wire Line
+	5350 4000 5350 2600
+Wire Wire Line
+	5350 2600 5250 2600
+Wire Wire Line
+	6000 3050 6000 3150
+Wire Wire Line
+	6000 3150 5550 3150
+Wire Wire Line
+	5550 3150 5550 2900
+Wire Wire Line
+	5550 2900 5250 2900
+Wire Wire Line
+	3350 3250 2350 3250
+Wire Wire Line
+	3450 3350 2350 3350
+Wire Wire Line
+	3450 2150 3450 3350
+Wire Wire Line
+	3350 2050 3350 3250
+$Comp
+L LP2950-3.0_TO92 U1
+U 1 1 5CABB898
+P 4950 1700
+F 0 "U1" H 4800 1825 50  0000 C CNN
+F 1 "LP2950-3.0_TO92" H 4950 1825 50  0000 L CNN
+F 2 "TO_SOT_Packages_THT:TO-92_Inline_Wide" H 4950 1925 50  0001 C CIN
+F 3 "" H 4950 1650 50  0001 C CNN
+	1    4950 1700
+	1    0    0    -1
+$EndComp
+$Comp
+L CP C1
+U 1 1 5BBB776B
+P 4700 2150
+F 0 "C1" H 4725 2250 50  0000 L CNN
+F 1 "CP" H 4725 2050 50  0000 L CNN
+F 2 "Capacitors_THT:CP_Radial_Tantal_D5.5mm_P5.00mm" H 4738 2000 50  0001 C CNN
+F 3 "" H 4700 2150 50  0001 C CNN
+	1    4700 2150
+	0    -1   -1   0
+$EndComp
+Wire Wire Line
+	4550 1700 4550 2150
+Wire Wire Line
+	4950 2000 4950 2250
+Wire Wire Line
+	4850 2150 5000 2150
+Connection ~ 4950 2150
+Wire Wire Line
+	5300 2150 5350 2150
+Connection ~ 5350 2150
+Wire Wire Line
+	5700 3050 5700 2750
+Wire Wire Line
+	5700 2750 6100 2750
+Wire Wire Line
+	5750 2650 6100 2650
+Wire Wire Line
+	3350 2050 3300 2050
+Wire Wire Line
 	3400 2550 3400 1750
 Wire Wire Line
-	3400 1750 3800 1750
-Wire Wire Line
-	3300 2450 3550 2450
-Wire Wire Line
-	3550 2450 3550 2200
-Wire Wire Line
-	3550 2200 3800 2200
-Wire Wire Line
-	3300 2350 3500 2350
-Wire Wire Line
-	3500 2350 3500 2650
-Wire Wire Line
-	3500 2650 3800 2650
-Wire Wire Line
-	6100 2550 6050 2550
-Wire Wire Line
-	6050 2550 6050 2400
-Wire Wire Line
-	6050 2100 6050 2050
-Wire Wire Line
-	6050 1750 6050 1650
-Wire Wire Line
-	5750 3250 4350 3250
-Wire Wire Line
-	6000 3050 6100 3050
-Wire Wire Line
-	5650 2950 6100 2950
-Wire Wire Line
-	5250 2800 5900 2800
-Wire Wire Line
-	5900 2850 6100 2850
-Wire Wire Line
-	5900 2800 5900 2850
-Wire Wire Line
-	5750 3250 5750 2750
-Wire Wire Line
-	5750 2750 6100 2750
-Wire Wire Line
-	5350 2500 4600 2500
-Wire Wire Line
-	4600 2500 4600 2700
-Wire Wire Line
-	4600 2700 4750 2700
-Wire Wire Line
-	5350 1750 5350 2500
-Wire Wire Line
-	4350 3250 4350 2800
-Wire Wire Line
-	4350 2800 4750 2800
-Wire Wire Line
-	6100 2650 5700 2650
-Wire Wire Line
-	5700 2650 5700 3050
-Wire Wire Line
-	5700 3050 4750 3050
-Wire Wire Line
-	4750 3050 4750 2900
-Wire Wire Line
-	5650 2950 5650 2700
-Wire Wire Line
-	5650 2700 5250 2700
-Wire Wire Line
-	6500 4000 5350 4000
-Wire Wire Line
-	5350 4000 5350 2600
-Wire Wire Line
-	5350 2600 5250 2600
-Wire Wire Line
-	6000 3050 6000 3150
-Wire Wire Line
-	6000 3150 5550 3150
-Wire Wire Line
-	5550 3150 5550 2900
-Wire Wire Line
-	5550 2900 5250 2900
-Wire Wire Line
-	2350 3250 3350 3250
-Wire Wire Line
-	2350 3350 3450 3350
-Wire Wire Line
-	3300 2250 3450 2250
-Wire Wire Line
-	3450 2250 3450 3350
-Wire Wire Line
-	3350 3250 3350 2150
-Wire Wire Line
-	3350 2150 3300 2150
+	3450 2150 3300 2150
+$Comp
+L Earth #PWR?
+U 1 1 5CABEB6C
+P 4950 2250
+F 0 "#PWR?" H 4950 2000 50  0001 C CNN
+F 1 "Earth" H 4950 2100 50  0001 C CNN
+F 2 "" H 4950 2250 50  0001 C CNN
+F 3 "" H 4950 2250 50  0001 C CNN
+	1    4950 2250
+	1    0    0    -1
+$EndComp
 $EndSCHEMATC
